File: circuit/pizzaTime.sch (KiCad schematic (older format))
At the start: 8 parts

Commit message: Updated circuit schematic
Parts:
- removed D? (x3): LED, symbol Device:LED
- removed R? (x3): R_PHOTO, symbol Device:R_PHOTO
- removed SW?: SW_MEC_5G, symbol Switch:SW_MEC_5G
- added C? (x3): CAP, symbol pspice:CAP
- added D? (x3): LED, symbol Device:LED
- added R? (x3): R_PHOTO, symbol Device:R_PHOTO
- added SW?: SW_Push, symbol Switch:SW_Push
Connections:
- net labels added: 1, RaspberryPiInterface
- net labels removed: +5V
- wire segments 36 -> 59
